Commit message: update guardian_description

File: trunk/guardian/guardian_sim/guardian_description/urdf/guardian.urdf (robot description, URDF)
Before this commit: robot guardian, 9 links, 8 joints
Links:
- added link left_track, mass 1.250; collision mesh filename=package://guardian_description/meshes/track.mesh; visual mesh filename=package://guardian_description/meshes/track.mesh
- added link right_track, mass 1.250; collision mesh filename=package://guardian_description/meshes/track.mesh; visual mesh filename=package://guardian_description/meshes/track.mesh
- link back_left_wheel: geometry collision mesh filename=package://guardian_description/meshes/wheel.mesh; visual mesh filename=package://guardian_description/meshes/wheel.mesh
- link back_right_wheel: geometry collision mesh filename=package://guardian_description/meshes/wheel.mesh; visual mesh filename=package://guardian_description/meshes/wheel.mesh
- link base_link: geometry collision box size=1.0 0.4 0.2; visual mesh filename=package://guardian_description/meshes/chassis.mesh
- link front_left_wheel: geometry collision mesh filename=package://guardian_description/meshes/wheel.mesh; visual mesh filename=package://guardian_description/meshes/wheel.mesh
- link front_right_wheel: geometry collision mesh filename=package://guardian_description/meshes/wheel.mesh; visual mesh filename=package://guardian_description/meshes/wheel.mesh
Joints:
- added joint joint_left_track: type fixed, parent base_link, child left_track, origin xyz=0.0 0.0 0.0 rpy=0 0 0
- added joint joint_right_track: type fixed, parent base_link, child right_track, origin xyz=0.0 0.0 0.0 rpy=0 0 3.1415926535
- joint joint_back_left_wheel: origin xyz=-0.30 0.25 0 rpy=0 0 0 -> xyz=-0.30 0.265 0 rpy=0 0 0
- joint joint_back_right_wheel: origin xyz=-0.30 -0.25 0 rpy=0 0 0 -> xyz=-0.30 -0.265 0 rpy=0 0 0
- joint joint_front_left_wheel: origin xyz=0.30 0.25 0 rpy=0 0 0 -> xyz=0.30 0.265 0 rpy=0 0 0
- joint joint_front_right_wheel: origin xyz=0.30 -0.25 0 rpy=0 0 0 -> xyz=0.30 -0.265 0 rpy=0 0 0

File: trunk/guardian/guardian_sim/guardian_description/urdf/guardian_without_controller.urdf (robot description, URDF)
Before this commit: robot guardian, 9 links, 8 joints
Links:
- added link left_track, mass 1.250; collision mesh filename=package://guardian_description/meshes/track.mesh; visual mesh filename=package://guardian_description/meshes/track.mesh
- added link right_track, mass 1.250; collision mesh filename=package://guardian_description/meshes/track.mesh; visual mesh filename=package://guardian_description/meshes/track.mesh
- link back_left_wheel: geometry collision mesh filename=package://guardian_description/meshes/wheel.mesh; visual mesh filename=package://guardian_description/meshes/wheel.mesh
- link back_right_wheel: geometry collision mesh filename=package://guardian_description/meshes/wheel.mesh; visual mesh filename=package://guardian_description/meshes/wheel.mesh
- link base_link: geometry collision box size=0.1 0.1 0.1; visual mesh filename=package://guardian_description/meshes/chassis.mesh
- link front_left_wheel: geometry collision mesh filename=package://guardian_description/meshes/wheel.mesh; visual mesh filename=package://guardian_description/meshes/wheel.mesh
- link front_right_wheel: geometry collision mesh filename=package://guardian_description/meshes/wheel.mesh; visual mesh filename=package://guardian_description/meshes/wheel.mesh
- link hokuyo_laser_box_link: geometry collision box size=0.05 0.05 0.1; visual box size=0.05 0.05 0.1
Joints:
- added joint joint_left_track: type fixed, parent base_link, child left_track, origin xyz=0.0 0.0 0.0 rpy=0 0 0
- added joint joint_right_track: type fixed, parent base_link, child right_track, origin xyz=0.0 0.0 0.0 rpy=0 0 3.1415926535
- joint joint_back_left_wheel: origin xyz=-0.30 0.25 0 rpy=0 0 0 -> xyz=-0.30 0.265 0 rpy=0 0 0
- joint joint_back_right_wheel: origin xyz=-0.30 -0.25 0 rpy=0 0 0 -> xyz=-0.30 -0.265 0 rpy=0 0 0
- joint joint_front_left_wheel: origin xyz=0.30 0.25 0 rpy=0 0 0 -> xyz=0.30 0.265 0 rpy=0 0 0
- joint joint_front_right_wheel: origin xyz=0.30 -0.25 0 rpy=0 0 0 -> xyz=0.30 -0.265 0 rpy=0 0 0
