Commit message: updated gwam_description with new mesh descriptions of the Guardian

File: trunk/gwam/gwam_sim/gwam_description/urdf/gwam.urdf (robot description, URDF)
Before this commit: robot guardian, 27 links, 26 joints
Links:
- added link left_track, mass 1.250; collision mesh filename=package://gwam_description/meshes/track.mesh; visual mesh filename=package://gwam_description/meshes/track.mesh
- added link right_track, mass 1.250; collision mesh filename=package://gwam_description/meshes/track.mesh; visual mesh filename=package://gwam_description/meshes/track.mesh
Joints:
- added joint joint_left_track: type fixed, parent base_link, child left_track, origin xyz=0.0 0.0 0.0 rpy=0 0 0
- added joint joint_right_track: type fixed, parent base_link, child right_track, origin xyz=0.0 0.0 0.0 rpy=0 0 3.1415926535
- joint joint_back_left_wheel: origin xyz=-0.30 0.25 0 rpy=0 0 0 -> xyz=-0.30 0.265 0 rpy=0 0 0
- joint joint_back_right_wheel: origin xyz=-0.30 -0.25 0 rpy=0 0 0 -> xyz=-0.30 -0.265 0 rpy=0 0 0
- joint joint_front_left_wheel: origin xyz=0.30 0.25 0 rpy=0 0 0 -> xyz=0.30 0.265 0 rpy=0 0 0
- joint joint_front_right_wheel: origin xyz=0.30 -0.25 0 rpy=0 0 0 -> xyz=0.30 -0.265 0 rpy=0 0 0

Commit message: update gwam.urdf

File: trunk/gwam/gwam_sim/gwam_description/urdf/gwam.urdf (robot description, URDF)
Before this commit: robot guardian, 29 links, 28 joints
Links:
- link base_link: mass 70.0 -> 85.0
Joints:
- joint base_footprint_joint: origin xyz=0 0 0.130 rpy=0 0 0 -> xyz=0 0 0.18 rpy=0 0 0
- joint wam_basejoint: origin xyz=0.0 -0.14 0.24 rpy=0 0 0 -> xyz=-0.060 -0.140 0.206 rpy=0 0 0
