Commit message: Adding gwam_common stack to repository, this contains gwam_bringup for launching scripts on multiple machines.

File: trunk/wam/wam_sim/wam_description/urdf/wam_4dof.urdf (robot description, URDF)
Before this commit: robot wam, 7 links, 6 joints
Links:
- removed link world
- added link wam_origin
Joints:
- joint wam_base_joint: parent world -> wam_origin

File: trunk/wam/wam_sim/wam_description/xacro/wam_4dof.urdf.xacro (robot description, xacro)
@@ -4,5 +4,5 @@
        xmlns:interface="http://playerstage.sourceforge.net/gazebo/xmlschema/#interface"
        xmlns:xacro="http://ros.org/wiki/xacro"
-       name="wam">
+       name="wam_4dof">
   <!-- LINKS   -->
   <include filename="$(find wam_description)/xacro/wam_base.urdf.xacro" />

File: trunk/wam/wam_sim/wam_description/xacro/wam_base.urdf.xacro (robot description, xacro)
@@ -2,5 +2,5 @@
 <robot xmlns:xacro="http://www.ros.org/wiki/xacro">
   <xacro:macro name="wam_base">
-    <link name="world"/>
+    <link name="wam_origin"/>
     <link name="wam_base">
         <inertial>
@@ -31,5 +31,5 @@
     </gazebo>
     <joint name="wam_base_joint" type="fixed">
-        <parent link="world"/>
+        <parent link="wam_origin"/>
         <child link="wam_base"/>
         <origin xyz="0.0 0.0 0.0" rpy="0 0 0" />
